Commit message: fix: bind MoveIt tool frame to source model

File: reference/mobile-manipulator/ros2_ws/src/jx_mobile_manipulator_moveit_config/config/reference_mobile_manipulator.urdf (robot description, URDF)
Before this commit: robot reference_mobile_manipulator, 7 links, 6 joints
Links:
- added link tool0
Joints:
- added joint tool0_fixed: type fixed, parent arm_link_6, child tool0, origin xyz=0.10 0 0 rpy=0 0 0

Commit message: release: prepare v0.5 simulation evidence

File: reference/mobile-manipulator/ros2_ws/src/jx_mobile_manipulator_moveit_config/config/reference_mobile_manipulator.urdf (robot description, URDF)
Before this commit: robot reference_mobile_manipulator, 8 links, 7 joints
Links:
- link arm_link_1: geometry collision cylinder length=0.18 radius=0.09; visual cylinder length=0.18 radius=0.09
- link arm_link_2: geometry collision cylinder length=0.35 radius=0.075; visual cylinder length=0.35 radius=0.075
- link arm_link_3: geometry collision cylinder length=0.30 radius=0.065; visual cylinder length=0.30 radius=0.065
- link arm_link_4: geometry collision cylinder length=0.20 radius=0.055; visual cylinder length=0.20 radius=0.055
- link arm_link_5: geometry collision cylinder length=0.12 radius=0.045; visual cylinder length=0.12 radius=0.045
- link arm_link_6: geometry collision cylinder length=0.10 radius=0.04; visual cylinder length=0.10 radius=0.04
- link base_link: geometry collision box size=0.8 0.6 0.4; visual box size=0.8 0.6 0.4
